Commit message: WIP [parsing] Add unit test files stolen from PR 16727
As of today (6e0f68619af253d6cd5fe762566956233ba1514a).

File: multibody/parsing/test/sdf_parser_test/interface_api_test/arm.urdf (robot description, URDF)
Before this commit: robot arm, 2 links, 1 joints
Links:
- link L1: geometry collision sphere radius=0.4; visual box size=0.1 0.1 0.1
