Commit message: [wsg_50_description] Refactor source control to use xacro

File: manipulation/models/wsg_50_description/sources/schunk_wsg_50.xacro (robot description, xacro)
@@ -1,9 +1,12 @@
-<?xml version="1.0" ?>
-<!-- =================================================================================== -->
-<!-- |    This document was autogenerated by xacro from manipulation/models/wsg_50_description/sources/schunk_wsg_50.sdf.xacro | -->
-<!-- |    EDITING THIS FILE BY HAND IS NOT RECOMMENDED                                 | -->
-<!-- =================================================================================== -->
-<sdf version="1.7" xmlns:drake="http://drake.mit.edu">
+<?xml version="1.0"?>
+<robot xmlns:xacro="http://ros.org/wiki/xacro">
+<xacro:macro name="schunk_gripper" params="with_ball_contact">
   <model name="Schunk_Gripper">
+    <xacro:if value="${with_ball_contact}">
+    <!--To enable faster simulation, the collision geometry in this model
+         consists of multiple spheres. These are arranged in a line along each
+         finger, with two additional spheres forming a triangle at each finger
+         tip.-->
+    </xacro:if>
     <link name="body">
       <pose>0 -0.049133 0 0 0 0</pose>
@@ -290,3 +293,4 @@
     <static>0</static>
   </model>
-</sdf>
+</xacro:macro>
+</robot>
